File: hardware/tablet.sch (EAGLE design)
At the start: 0 parts

Commit message: Initial analog front end schematic
Parts:
- added C1: ~470pF, 0jpe:C0603
- added C2, C3, C4, C5, C6, C7: 100nF, 0jpe:C0603
- added D1: BAT721S, 0jpe:D2_SERIESSOT23
- added D2: 3V9, 0jpe:DSOD323
- added IC1: (no value), 0jpe:OPAMP_DUALSOIC8
- added IC2: MCP3201, 0jpe:MCP3201
- added IC3: DG9233EDY, 0jpe:DG9233EDY
- added IC4: MAX6104EUR, 0jpe:MAX6104EUR
- added R1: TBD, 0jpe:R0603
- added R2, R3: 1K, 0jpe:R0603
Connections:
- new net +5V: C2.1, C4.1, C5.1, C7.1, IC1PWR.V+, IC2.VDD, IC3PWR.V+, IC4.VIN
- new net -5V: C3.2, IC1PWR.V-
- new net ADC_CS: IC2.!CS!/SHDN
- new net GND: C2.2, C3.1, C4.2, C5.2, C6.2, C7.2, IC1A.-IN, IC1B.+IN, IC2.IN-, IC2.VSS, IC3PWR.V-, IC4.GND
- new net INT_EN: IC3A.SEL
- new net INT_RST: IC3B.SEL
- new net MISO: IC2.DOUT
- new net N$1: D1.A, IC3A.COM, R1.2
- new net N$2: D1.C, IC1A.+IN, R1.1, R2.2
- new net N$3: D1.COM, IC1A.OUT
- new net N$4: C1.2, D2.1, IC1B.-IN, IC3B.COM, R3.2
- new net N$6: C6.1, IC2.VREF, IC4.VOUT
- new net N$7: IC3A.NO, R3.1
- new net SCLK: IC2.CLK
- new net SIG: R2.1
- new net VOUT: C1.1, D2.2, IC1B.OUT, IC2.IN+, IC3B.NO
